File: schematics/stm32_devboard.kicad_sch (KiCad schematic)
At the start: 15 parts, among them J1 Conn_ARM_JTAG_SWD_10, J2 USB_C_Receptacle_USB2.0_14P, SW1 SW_Push, SW2 SW_Push, U1 STM32F401RETx, U2 AP2112K-3.3

Commit message: Update PCB layout progress
Parts:
- added C10, C11, C12: 100n, Capacitor_SMD:C_0603_1608Metric, symbol Device:C
- added C13: 4.7u, Capacitor_SMD:C_0603_1608Metric, symbol Device:C
- added C6, C7: 1u, Capacitor_SMD:C_0603_1608Metric, symbol Device:C
- added C8, C9: 22p, Capacitor_SMD:C_0603_1608Metric, symbol Device:C
- added D2: LED, LED_SMD:LED_0603_1608Metric, symbol Device:LED
- added J3: Conn_01x16, Connector_PinHeader_2.54mm:PinHeader_2x08_P2.54mm_Vertical, symbol Connector_Generic:Conn_01x16
- added R4: 1K, Resistor_SMD:R_0603_1608Metric, symbol Device:R
- added Y1: 8 MHz, Crystal:Crystal_SMD_3225-4Pin_3.2x2.5mm, symbol Device:Crystal
- C1: footprint (none) -> Capacitor_SMD:C_0805_2012Metric
- C2, C4, C5: footprint (none) -> Capacitor_SMD:C_0603_1608Metric
- C3: value C -> 100n; footprint (none) -> Capacitor_SMD:C_0603_1608Metric
- D1: footprint (none) -> LED_SMD:LED_0603_1608Metric
- J1: footprint (none) -> Connector_PinHeader_2.54mm:PinHeader_2x05_P2.54mm_Vertical
- J2: footprint (none) -> Connector_USB:USB_C_Receptacle_JAE_DX07S024WJ3R400
- R1, R2: footprint (none) -> Resistor_SMD:R_0603_1608Metric
- R3: value R -> 330; footprint (none) -> Resistor_SMD:R_0603_1608Metric
- SW1, SW2: footprint (none) -> Button_Switch_SMD:SW_SPST_TL3342
Connections:
- net +3.3V: now also C3.1, U1.1 (VBAT), C10.1, C11.1, C12.1, C13.1, C7.1, J3.15 (Pin_15), R4.1; no longer C3.2
- net GND: now also C3.2, C10.2, C11.2, C12.2, C13.2, C7.2, C8.2, C9.2, D2.1 (K), J3.16 (Pin_16); no longer C3.1
- net USER_BUTTON: now also J3.7 (Pin_7)
- net USER_LED: now also J3.6 (Pin_6)
- net at J2.A4 (VBUS), J2.A9 (VBUS), J2.B4 (VBUS)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: now also C6.1; no longer U2.1 (VIN), U2.3 (EN)
- net at U1.14 (PA0): now also J3.1 (Pin_1)
- net at U1.15 (PA1): now also J3.2 (Pin_2)
- net at U1.16 (PA2): now also J3.3 (Pin_3)
- net at U1.17 (PA3): now also J3.4 (Pin_4)
- net at U1.20 (PA4): now also J3.5 (Pin_5)
- net at U1.23 (PA7): now also J3.8 (Pin_8)
- net at U1.26 (PB0): now also J3.9 (Pin_9)
- net at U1.27 (PB1): now also J3.10 (Pin_10)
- net at U1.5 (PH0): now also C8.1, Y1.2
- net at U1.58 (PB6): now also J3.11 (Pin_11)
- net at U1.59 (PB7): now also J3.12 (Pin_12)
- net at U1.6 (PH1): now also C9.1, Y1.1
- net at U1.61 (PB8): now also J3.13 (Pin_13)
- net at U1.62 (PB9): now also J3.14 (Pin_14)
- new net: C6.2, U2.1 (VIN), U2.3 (EN)
- new net: D2.2 (A), R4.2
- no-connect marks 0 -> 39
Other:
- note added: "power section"
- note added: "swd"
- moved on the sheet: C4, C5, J2, U2
